Commit message: Gazebo world ortamı eklendi, robot sürtünme problemi ortadan kaldırıldı.

File: src/my_robot_description/urdf/lidar.xacro (robot description, xacro)
@@ -7,14 +7,14 @@
         <visual>
             <geometry>
-                <cylinder radius="${lidar_radius}" length="${lidar_length"/>
+                <cylinder radius="${lidar_radius}" length="${lidar_length}"/>
             </geometry>
-            <origin xyz="0 0 0" rpy="$0 0 0"/>
+            <origin xyz="0 0 0" rpy="0 0 0"/>
             <material name="grey"/>
         </visual>
         <collision>
             <geometry>
-                <cylinder radius="${lidar_radius}" length="${lidar_length"/>
+                <cylinder radius="${lidar_radius}" length="${lidar_length}"/>
             </geometry>
-            <origin xyz="0 0 0" rpy="$0 0 0"/>
+            <origin xyz="0 0 0" rpy="0 0 0"/>
         </collision>
         <xacro:cylinder_inertia m = "0.2" r="${2*lidar_radius}"

File: src/my_robot_description/urdf/properties_gazebo.xacro (robot description, xacro)
@@ -12,4 +12,6 @@
     <gazebo reference = "caster_wheel_link">
         <material>Gazebo/Black</material>
+        <mu1 value="0.1"/>
+        <mu2 value = "0.1"/>
     </gazebo>
     <gazebo>
